File: ereader/ereader_rev1.kicad_sch (KiCad schematic)
At the start: 0 parts

Commit message: WIP: integrate orientation sensor and refresh schematic review exports
Add LIS2DW12 host wiring and sourced passives, revise held-supply discharge calculations, document camera and capacitance screens, and refresh standard capacitor caches. Include reviewed 14-page PDF and reconciled native BOM. ERC remains 111 errors and 11 warnings; electrical design is incomplete. Refs #21.
Other:
- added sheet Orientation sensor (orientation_sensor.kicad_sch)
- sheet RA8P1 IO allocation ports: added SENS_INT1, SENS_SCL, SENS_SDA; removed none
Changed lines of the file:
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@@
+	(wire
+		(pts
+			(xy 199.39 120.65) (xy 207.01 120.65)
+		)
+		(stroke
+			(width 0)
+			(type default)
+		)
+	)
 	(wire
 		(pts
@@
 	(wire
 		(pts
+			(xy 199.39 128.27) (xy 207.01 128.27)
+		)
+		(stroke
+			(width 0)
+			(type default)
+		)
+	)
+	(wire
+		(pts
 			(xy 209.55 186.69) (xy 209.55 104.14)
 		)
@@
 	(wire
 		(pts
+			(xy 429.26 189.23) (xy 441.96 189.23)
+		)
+		(stroke
+			(width 0)
+			(type default)
+		)
+	)
+	(wire
+		(pts
 			(xy 52.07 87.63) (xy 62.23 87.63)
 		)
@@
 	(wire
 		(pts
+			(xy 429.26 186.69) (xy 441.96 186.69)
+		)
+		(stroke
+			(width 0)
+			(type default)
+		)
+	)
+	(wire
+		(pts
 			(xy 91.44 73.66) (xy 91.44 77.47)
 		)
@@
 	(wire
 		(pts
+			(xy 556.26 186.69) (xy 568.96 186.69)
+		)
+		(stroke
+			(width 0)
+			(type default)
+		)
+	)
+	(wire
+		(pts
 			(xy 127 133.35) (xy 127 140.97)
 		)
@@
 		(pts
 			(xy 102.87 133.35) (xy 102.87 140.97)
+		)
+		(stroke
+			(width 0)
+			(type default)
+		)
+	)
+	(wire
+		(pts
+			(xy 199.39 113.03) (xy 207.01 113.03)
 		)
 		(stroke
@@
 		)
 	)
+	(label "SENS_SDA"
+		(at 207.01 128.27 180)
+		(effects
+			(font
+				(size 1.27 1.27)
+			)
+			(justify right bottom)
+		)
+	)
 	(label "SDRAM_WE_N"
 		(at 379.73 133.35 0)
@@
 		)
 	)
+	(label "SENS_INT1"
+		(at 568.96 186.69 0)
+		(effects
+			(font
+				(size 1.27 1.27)
+			)
+			(justify left bottom)
+		)
+	)
 	(label "SD_CMD"
 		(at 318.77 257.81 0)
@@
 		)
 	)
+	(label "SENS_SDA"
+		(at 429.26 189.23 0)
+		(effects
+			(font
+				(size 1.27 1.27)
+			)
+			(justify left bottom)
+		)
+	)
 	(label "SDRAM_CAS_N"
 		(at 379.73 143.51 0)
@@
 		)
 	)
+	(label "SENS_SCL"
+		(at 207.01 120.65 180)
+		(effects
+			(font
+				(size 1.27 1.27)
+			)
+			(justify right bottom)
+		)
+	)
 	(label "SD_PWR_REQ"
 		(at 104.14 73.66 90)
@@
 		)
 	)
+	(label "SENS_SCL"
+		(at 429.26 186.69 0)
+		(effects
+			(font
+				(size 1.27 1.27)
+			)
+			(justify left bottom)
+		)
+	)
 	(label "NOR_DS_HOST"
 		(at 55.88 52.07 180)
@@
 			)
 			(justify left bottom)
+		)
+	)
+	(label "SENS_INT1"
+		(at 207.01 113.03 180)
+		(effects
+			(font
+				(size 1.27 1.27)
+			)
+			(justify right bottom)
 		)
 	)
@@
 			)
 		)
+		(pin "SENS_INT1" input
+			(at 199.39 113.03 0)
+			(effects
+				(font
+					(size 1.27 1.27)
+				)
+				(justify right)
+			)
+		)
+		(pin "SENS_SCL" output
+			(at 199.39 120.65 0)
+			(effects
+				(font
+					(size 1.27 1.27)
+				)
+				(justify right)
+			)
+		)
+		(pin "SENS_SDA" bidirectional
+			(at 199.39 128.27 0)
+			(effects
+				(font
+					(size 1.27 1.27)
+				)
+				(justify right)
+			)
+		)
 		(instances
 			(project "ereader_rev1"
@@
 				)
 			)
+		)
+	)
+	(sheet
+		(at 441.96 184.15)
+		(size 114.3 44.45)
+		(exclude_from_sim no)
+		(in_bom yes)
+		(on_board yes)
+		(dnp no)
+		(fields_autoplaced yes)
+		(stroke
+			(width 0.1524)
+			(type solid)
+		)
+		(fill
+			(color 0 0 0 0)
+		)
+		(property "Sheetname" "Orientation sensor"
+			(at 441.96 183.4384 0)
+			(show_name no)
+			(do_not_autoplace no)
+			(effects
+				(font
+					(size 1.27 1.27)
+				)
+				(justify left bottom)
+			)
+		)
+		(property "Sheetfile" "orientation_sensor.kicad_sch"
+			(at 441.96 229.1846 0)
+			(show_name no)
+			(do_not_autoplace no)
+			(effects
+				(font
+					(size 1.27 1.27)
+				)
+				(justify left top)
+			)
+		)
+		(pin "SENS_SCL" input
+			(at 441.96 186.69 180)
+			(effects
+				(font
+					(size 1.27 1.27)
+				)
+				(justify left)
+			)
+		)
+		(pin "SENS_SDA" bidirectional
+			(at 441.96 189.23 180)
+			(effects
+				(font
+					(size 1.27 1.27)
+				)
+				(justify left)
+			)
+		)
+		(pin "SENS_INT1" output
+			(at 556.26 186.69 0)
+			(effects
+				(font
+					(size 1.27 1.27)
+				)
+				(justify right)
+			)
+		)
+		(instances
+			(project "ereader_rev1"
+				(path "/0586cc51-9c57-495b-a0c9-c29ba0d48166"
+					(page "14")
+				)
+			)
