File: ereader/mcu_core_power.kicad_sch (KiCad schematic)
At the start: 17 parts, among them U1 R7KA8P1KFLCAC#UC0

Commit message: WIP: integrate orientation sensor and refresh schematic review exports
Add LIS2DW12 host wiring and sourced passives, revise held-supply discharge calculations, document camera and capacitance screens, and refresh standard capacitor caches. Include reviewed 14-page PDF and reconciled native BOM. ERC remains 111 errors and 11 warnings; electrical design is incomplete. Refs #21.
Parts:
- C9: Selection_Basis Do not approve GRM32ER70J476KE20L solely from Renesas examp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 -> Candidate: Murata GRM32ER71A476KE15K, 47uF +/-10%, 10V X7R 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; Sourcing_Snapshot 2026-09-05 live Mouser search: GRM32ER70J476KE20L stock7034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 -> 2026-09-27 DigiKey page: candidate GRM32ER71A476KE15K Activ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
Changed lines of the file:
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@@
 			)
 		)
-		(property "Sourcing_Snapshot" "2026-09-05 live Mouser search: GRM32ER70J476KE20L stock7034, End of Life; DigiKey indexed stock0 Active (conflict)"
+		(property "Sourcing_Snapshot" "2026-09-27 DigiKey page: candidate GRM32ER71A476KE15K Active, 1595 unreserved, USD0.98 qty1 / 0.43690 qty100, 17wk. Earlier GRM32ER70J476KE20L lifecycle conflict retained in design/core_bulk_c9.md; not purchase approval."
 			(at 254 177.8 0)
 			(hide yes)
@@
 			)
 		)
-		(property "Selection_Basis" "Do not approve GRM32ER70J476KE20L solely from Renesas example: Mouser EOL flag; replacement and bias qualification required"
+		(property "Selection_Basis" "Candidate: Murata GRM32ER71A476KE15K, 47uF +/-10%, 10V X7R 1210. Murata GRM32ER71A476KE15-04CA (2025-01-10). HOLD pending DC-bias/aging and RA8P1 core-loop qualification; see design/core_bulk_c9.md."
 			(at 254 177.8 0)
 			(hide yes)
