File: ereader/mcu_interfaces.kicad_sch (KiCad schematic)
At the start: 10 parts, among them U1 R7KA8P1KFLCAC#UC0

Commit message: WIP: integrate orientation sensor and refresh schematic review exports
Add LIS2DW12 host wiring and sourced passives, revise held-supply discharge calculations, document camera and capacitance screens, and refresh standard capacitor caches. Include reviewed 14-page PDF and reconciled native BOM. ERC remains 111 errors and 11 warnings; electrical design is incomplete. Refs #21.
Connections:
- net SENS_INT1: now reaches U1.D11 (P306)
- net SENS_SCL: now reaches U1.K13 (P410)
- net SENS_SDA: now reaches U1.R16 (P409)
Changed lines of the file:
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@@
 	(wire
 		(pts
+			(xy 264.16 63.5) (xy 271.78 63.5)
+		)
+		(stroke
+			(width 0)
+			(type default)
+		)
+	)
+	(wire
+		(pts
 			(xy 210.82 132.08) (xy 233.68 132.08)
 		)
@@
 	(wire
 		(pts
+			(xy 317.5 71.12) (xy 330.2 71.12)
+		)
+		(stroke
+			(width 0)
+			(type default)
+		)
+	)
+	(wire
+		(pts
 			(xy 105.41 207.01) (xy 105.41 205.74)
 		)
@@
 	(wire
 		(pts
+			(xy 317.5 73.66) (xy 330.2 73.66)
+		)
+		(stroke
+			(width 0)
+			(type default)
+		)
+	)
+	(wire
+		(pts
 			(xy 132.08 127) (xy 137.16 127)
 		)
@@
 		)
 	)
+	(hierarchical_label "SENS_SCL"
+		(shape output)
+		(at 317.5 73.66 180)
+		(effects
+			(font
+				(size 1.27 1.27)
+			)
+			(justify right)
+		)
+	)
 	(hierarchical_label "POWER_BUTTON_N"
 		(shape input)
@@
 		)
 	)
+	(hierarchical_label "SENS_INT1"
+		(shape input)
+		(at 271.78 63.5 0)
+		(effects
+			(font
+				(size 1.27 1.27)
+			)
+			(justify left)
+		)
+	)
 	(hierarchical_label "CAM_CLK_P"
 		(shape input)
@@
 		)
 	)
+	(hierarchical_label "SENS_SDA"
+		(shape bidirectional)
+		(at 317.5 71.12 180)
+		(effects
+			(font
+				(size 1.27 1.27)
+			)
+			(justify right)
+		)
+	)
 	(hierarchical_label "CEU_D2"
 		(shape input)
@@
 		)
 		(pin "D11"
+			(alternate "IRQ28-DS")
 		)
 		(pin "C11"
@@
 		)
 		(pin "R16"
+			(alternate "SDA0_A")
 		)
 		(pin "K13"
+			(alternate "SCL0_A")
 		)
 		(pin "M14"
