File: ereader/mcu_interfaces.kicad_sch (KiCad schematic)
At the start: 10 parts, among them U1 R7KA8P1KFLCAC#UC0

Commit message: Add buffered SCI4 NAND storage schematic
Connections:
- net NAND_MOSI: now reaches U1.N14 (P714)
- net NAND_MISO: now reaches U1.T15 (P715)
- net NAND_CS_N: now reaches U1.P14 (P413)
- net NAND_SCK: now reaches U1.R14 (P514)
Changed lines of the file:
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@@
 	)
 	(wire (pts (xy 167.64 121.92) (xy 172.72 121.92)) (stroke (width 0) (type default)))
+(wire (pts (xy 360.68 83.82) (xy 382.27 83.82)) (stroke (width 0) (type default)))
+(hierarchical_label "NAND_SCK" (shape output) (at 382.27 83.82 0) (effects (font (size 1.27 1.27)) (justify left bottom)))
+(wire (pts (xy 330.2 81.28) (xy 308.61 81.28)) (stroke (width 0) (type default)))
+(hierarchical_label "NAND_CS_N" (shape output) (at 308.61 81.28 180) (effects (font (size 1.27 1.27)) (justify right bottom)))
+(wire (pts (xy 71.12 157.48) (xy 88.9 157.48)) (stroke (width 0) (type default)))
+(hierarchical_label "NAND_MOSI" (shape output) (at 88.9 157.48 0) (effects (font (size 1.27 1.27)) (justify left bottom)))
+(wire (pts (xy 71.12 160.02) (xy 88.9 160.02)) (stroke (width 0) (type default)))
+(hierarchical_label "NAND_MISO" (shape input) (at 88.9 160.02 0) (effects (font (size 1.27 1.27)) (justify left bottom)))
 )
