File: ereader/power_button.kicad_sch (KiCad schematic)
At the start: 37 parts, among them Q1 DMN2056U-7, Q2 DMN2056U-7, SW1 POWER, U10 LM66100DCKR, U11 TPS3808G01DBVR, U12 74LVC1G14GW,125, U9 LTC2954ITS8-1

Commit message: WIP: integrate orientation sensor and refresh schematic review exports
Add LIS2DW12 host wiring and sourced passives, revise held-supply discharge calculations, document camera and capacitance screens, and refresh standard capacitor caches. Include reviewed 14-page PDF and reconciled native BOM. ERC remains 111 errors and 11 warnings; electrical design is incomplete. Refs #21.
Parts:
- C63, C64, C65, C66: value 100u -> 220u; DigiKey_Part_Number 399-3769-1-ND -> 399-8379-1-ND; DigiKey_URL https://www.digikey.com/en/products/detail/kemet/T491D107K0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 -> https://www.digikey.com/en/products/detail/kemet/T491D227K0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; Manufacturer_Part_Number T491D107K010AT -> T491D227K010AT; Selection_Basis SYS-007 revised: four parallel 100uF/10V tantalum capacitor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 -> SENS-010 / SYS-007 revision: four parallel 220uF/10V. Cmin=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; Sourcing_Snapshot 2026-09-07: DigiKey Active, stock 11863; USD 1.64/1.09/0.80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 -> 2026-09-27: DigiKey Active; stock 3958 unreserved; USD2.24/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
- R31: Selection_Basis SYS-007 revised: 100R between U10 VOUT and AON_HOLD; CE sen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 -> SENS-010 / SYS-007 revision: 100R between U10 VOUT and AON_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
- R39, R40: Selection_Basis SYS-007 / PWR-004: two 22R 1W in parallel, Rpath_max=11.421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 -> SENS-010 / SYS-007 revision: two22R1W in parallel; Rpath_ma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
- U10: Selection_Basis SYS-007 revised: VIN1=raw SYS_AON, VOUT6 via R31=100R to AO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 -> SENS-010 / SYS-007 revision: VIN1=raw SYS_AON, VOUT6 via R3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
Other:
- note added: "SYS-007 / SENS-010: HELD SUPPLY / U10, R31, C62-C66 C63-C66: 4 x 220uF/10V; Cmin=880uF*0.9^3=641.52uF. VIN=raw SYS; VOUT->R31->reservoir; CE senses reservoir. Icontrol<=1.825mA incl 1.100mA bank leakage screen. Reverse allowance=0.817mA; Itotal<=2.642mA. Vinitial=3.263705831-max(0.250,1.825mA*102.24ohm) =3.013705831V; shared transition reserve=1uC. thold=[641.52uF*(Vinitial-2.7V)-1uC]/2.642mA =75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"
- note added: "SYS-007 / SENS-010: SHUTDOWN / U12, Q1-Q3, R35-R40, R70-R71 POWER_OFF_H=NOT(MAIN_PWR_EN); held-domain VCC=2.7..4.6V. Each gate branch: 1k series / 1M pulldown; 1% +100ppm/C, 100C. 4-gate peak<=4*4.6/(1000*0.99^2)=18.773595mA <50mA. Includes future USB-clear; static<=22.773595uA <100uA. VGSmin=(2.6-1020.1*1uA)/(1+1020.1/980100)=2.596278V. 1uA per gate/board leakage is a qualification allocation. R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"
- note removed: "SYS-007 / PWR-004: HELD SUPPLY / U10, R31, C62-C66 C63-C66: 4 x 100uF/10V; Cmin=400uF*0.9^3=291.6uF. VIN=raw SYS; VOUT->R31->reservoir; CE senses reservoir. Icontrol<=1.125mA incl 500uA bank leakage allocation. Pre-trip reverse: 80mV/98.01ohm<0.817mA. Itotal=1.942mA. Vinitial=3.263705831-max(0.250,0.001125*102.24) =3.013705831V (threshold OR resistive-drop limit). t_hold=[291.6uF*(3.013705831-2.7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"
- note removed: "SYS-007 / PWR-004: SHUTDOWN / U12, Q1-Q3, R35-R40, R70-R71 POWER_OFF_H=NOT(MAIN_PWR_EN); held-domain VCC=2.7..4.6V. Each gate branch: 1k series / 1M pulldown; 1% + 100ppm/C, 100C. 4-gate peak<=4*4.6/(1000*0.99^2)=18.773595mA <50mA. Includes future USB-clear; static<=22.773595uA <100uA. VGSmin=(2.6-1020.1*1uA)/(1+1020.1/980100)=2.596278V. 1uA per gate/board leakage is a qualification allocation. R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"
