File: ereader/radio_esp32.kicad_sch (KiCad schematic)
At the start: 38 parts, among them U25 TXU0102DCUR, U27 TXU0202DCUR, U3 ESP32-C6-WROOM-1-N8, U4 TPS22964CYZPT, U5 TXU0304PWR, U6 TPS389001DSET, U7 SN74LVC1G97DBVR, U8 SN74LVC1G97DBVR

Commit message: Add fixture UART input pull-up and refresh schematic PDF
Parts:
- added R107: 10k, symbol Device:R
Connections:
- net SERVICE_VIO: now also R107.1
- net SERVICE_TX: now reaches U27.5 (A1)
- net SERVICE_TX: now also R107.2
Changed lines of the file:
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@@
 	)
 	(junction
+		(at 96.52 306.07)
+		(diameter 0)
+		(color 0 0 0 0)
+	)
+	(junction
 		(at 228.6 109.22)
 		(diameter 0)
@@
 	(wire
 		(pts
+			(xy 96.52 306.07) (xy 124.46 306.07)
+		)
+		(stroke
+			(width 0)
+			(type default)
+		)
+	)
+	(wire
+		(pts
 			(xy 228.6 107.95) (xy 228.6 109.22)
 		)
@@
 	(wire
 		(pts
-			(xy 81.28 306.07) (xy 124.46 306.07)
+			(xy 81.28 306.07) (xy 96.52 306.07)
 		)
 		(stroke
@@
 	(wire
 		(pts
+			(xy 96.52 306.07) (xy 96.52 312.42)
+		)
+		(stroke
+			(width 0)
+			(type default)
+		)
+	)
+	(wire
+		(pts
 			(xy 134.62 154.94) (xy 142.24 154.94)
 		)
@@
 	(wire
 		(pts
+			(xy 96.52 320.04) (xy 96.52 328.93)
+		)
+		(stroke
+			(width 0)
+			(type default)
+		)
+	)
+	(wire
+		(pts
 			(xy 290.83 184.15) (xy 311.15 184.15)
 		)
@@
 	(wire
 		(pts
+			(xy 96.52 328.93) (xy 134.62 328.93)
+		)
+		(stroke
+			(width 0)
+			(type default)
+		)
+	)
+	(wire
+		(pts
 			(xy 170.18 306.07) (xy 170.18 309.88)
 		)
@@
 		)
 	)
+	(label "SERVICE_TX"
+		(at 111.76 328.93 0)
+		(effects
+			(font
+				(size 1.27 1.27)
+			)
+			(justify left bottom)
+		)
+	)
 	(label "C6_GPIO15"
 		(at 137.16 87.63 0)
@@
 					(unit 1)
 				)
+			)
+		)
+	)
+	(symbol
+		(lib_id "Device:R")
+		(at 96.52 316.23 0)
+		(unit 1)
+		(body_style 1)
+		(exclude_from_sim no)
+		(in_bom yes)
+		(on_board yes)
+		(in_pos_files yes)
+		(dnp no)
+		(property "Reference" "R107"
+			(at 100.33 314.96 0)
+			(show_name no)
+			(do_not_autoplace no)
+			(effects
+				(font
+					(size 1.27 1.27)
+				)
+				(justify left)
+			)
+		)
+		(property "Value" "10k"
+			(at 100.33 317.5 0)
+			(show_name no)
+			(do_not_autoplace no)
+			(effects
+				(font
+					(size 1.27 1.27)
+				)
+				(justify left)
+			)
+		)
+		(property "Footprint" ""
+			(at 94.742 316.23 0)
+			(hide yes)
+			(show_name no)
+			(do_not_autoplace no)
+			(effects
+				(font
+					(size 1.27 1.27)
+				)
+			)
+		)
+		(property "Datasheet" "https://www.yageogroup.com/component-documentation/download/specsheet/RC0603FR-0710KL"
+			(at 96.52 316.23 0)
+			(hide yes)
+			(show_name no)
+			(do_not_autoplace no)
+			(effects
+				(font
+					(size 1.27 1.27)
+				)
+			)
+		)
+		(property "Description" "YAGEO RC0603FR-0710KL; 10k, 1%, 100 ppm/C; U27 UART input idle-high pull-up to its local supply. SERVICE-004/005 conditional screen; leakage and sequencing qualification pending."
+			(at 96.52 316.23 0)
+			(hide yes)
+			(show_name no)
+			(do_not_autoplace no)
+			(effects
+				(font
+					(size 1.27 1.27)
+				)
+			)
+		)
+		(property "ki_keywords" "R res resistor"
+			(at 96.52 316.23 0)
+			(hide yes)
+			(show_name no)
+			(do_not_autoplace no)
+			(effects
+				(font
+					(size 1.27 1.27)
+				)
+			)
+		)
+		(property "ki_fp_filters" "R_*"
+			(at 96.52 316.23 0)
+			(hide yes)
+			(show_name no)
+			(do_not_autoplace no)
+			(effects
+				(font
+					(size 1.27 1.27)
+				)
+			)
+		)
+		(property "DigiKey_Part_Number" "311-10.0KHRCT-ND"
+			(at 96.52 316.23 0)
+			(hide yes)
+			(show_name no)
+			(do_not_autoplace no)
+			(effects
+				(font
+					(size 1.27 1.27)
+				)
+			)
+		)
+		(property "DigiKey_URL" "https://www.digikey.com/en/products/detail/yageo/RC0603FR-0710KL/729827"
+			(at 96.52 316.23 0)
+			(hide yes)
+			(show_name no)
+			(do_not_autoplace no)
+			(effects
+				(font
+					(size 1.27 1.27)
+				)
+			)
+		)
+		(property "Procurement_Status" "Selected for U27 UART input idle-high pull-up to its local supply; installed leakage and sequencing qualification pending; footprint deferred."
+			(at 96.52 316.23 0)
+			(hide yes)
+			(show_name no)
+			(do_not_autoplace no)
+			(effects
+				(font
+					(size 1.27 1.27)
+				)
+			)
+		)
+		(property "Sourcing_Snapshot" "2026-09-05 indexed: stock 2922248; Active; USD CT 1:0.10 / 10:0.025 / 100:0.01220 / 1000:0.00661; 17wk lead; recheck before order"
+			(at 96.52 316.23 0)
+			(hide yes)
+			(show_name no)
+			(do_not_autoplace no)
+			(effects
+				(font
+					(size 1.27 1.27)
+				)
+			)
+		)
+		(property "Manufacturer_Name" "YAGEO"
+			(at 96.52 316.23 0)
+			(hide yes)
+			(show_name no)
+			(do_not_autoplace no)
+			(effects
+				(font
+					(size 1.27 1.27)
+				)
+			)
+		)
+		(property "Manufacturer_Part_Number" "RC0603FR-0710KL"
+			(at 96.52 316.23 0)
+			(hide yes)
+			(show_name no)
+			(do_not_autoplace no)
+			(effects
+				(font
+					(size 1.27 1.27)
+				)
+			)
+		)
+		(property "Selection_Basis" "SERVICE-004/005: 10k pull-up on U27 A1 or B2 to the corresponding VCCA or VCCB supply. R=9801..10201 ohm under 1% tolerance and 1% temperature allocation. Conditional DC screen only; installed leakage, adapter and sequencing qualification pending."
+			(at 96.52 316.23 0)
+			(hide yes)
+			(show_name no)
+			(do_not_autoplace no)
+			(effects
+				(font
+					(size 1.27 1.27)
+				)
+			)
+		)
+		(property "Mouser_URL" ""
+			(at 96.52 316.23 0)
+			(hide yes)
+			(show_name no)
+			(do_not_autoplace no)
+			(effects
+				(font
+					(size 1.27 1.27)
+				)
+			)
+		)
+		(pin "1"
+		)
+		(pin "2"
+		)
+		(instances
+			(project "ereader_rev1"
+				(path "/0586cc51-9c57-495b-a0c9-c29ba0d48166/9b84c337-6879-4714-899e-3993bcc30b88"
+					(reference "R107")
+					(unit 1)
+				)
